File: Final Project KiCAD designs/Final Project KiCAD designs.kicad_sch (KiCad schematic)
At the start: 28 parts, among them J1 Conn_02x08_Counter_Clockwise, J2 Jack-DC, U1 74HC595, U2 74HC595, U3 HDSP-A151, U4 HDSP-A151

Commit message: PCB Designs and Sound
Parts:
- added J3, J4: Screw_Terminal_01x02, TerminalBlock:TerminalBlock_bornier-2_P5.08mm, symbol Connector:Screw_Terminal_01x02
- added R15: 10kR, Resistor_THT:R_Axial_DIN0207_L6.3mm_D2.5mm_P7.62mm_Horizontal, symbol Device:R
- added SW1: SW_Push, Button_Switch_THT:SW_PUSH-12mm_Wuerth-430476085716, symbol Switch:SW_Push
- BZ1: footprint (none) -> Buzzer_Beeper:Buzzer_TDK_PS1240P02BT_D12.2mm_H6.5mm
- C1: footprint (none) -> Capacitor_THT:CP_Radial_D8.0mm_P3.80mm
- C2: footprint (none) -> Capacitor_THT:C_Disc_D4.7mm_W2.5mm_P5.00mm
- J1: value Conn_02x08_Counter_Clockwise -> LED_Matrix_Header; footprint (none) -> Connector_PinHeader_2.54mm:PinHeader_2x08_P2.54mm_Vertical
- J2: footprint (none) -> Connector_BarrelJack:BarrelJack_Horizontal
- R1, R10, R11, R12, R13, R14, R2, R3, R4, R5, R6, R7, R8, R9: footprint (none) -> Resistor_THT:R_Axial_DIN0207_L6.3mm_D2.5mm_P7.62mm_Horizontal
- RV1, RV2: footprint (none) -> Connector_PinHeader_2.54mm:PinHeader_1x03_P2.54mm_Horizontal
- U1, U2: footprint (none) -> Package_DIP:DIP-16_W7.62mm
Connections:
- net +5V: now also J3.1 (Pin_1), J3.2 (Pin_2), R15.1
- net GND: now also A2.29 (GND), A2.4 (GND), J1.11 (Pin_11), J1.13 (Pin_13), J1.15 (Pin_15), J1.9 (Pin_9), J4.1 (Pin_1), J4.2 (Pin_2), SW1.2
- net R0: now reaches J1.1 (Pin_1)
- net R0: now also A2.5 (D2)
- net LAT: now reaches J1.10 (Pin_10)
- net LAT: now also A2.13 (D10)
- net RowB: now reaches J1.12 (Pin_12)
- net RowB: now also A2.20 (A1)
- net G1: now reaches J1.14 (Pin_14)
- net G1: now also A2.9 (D6)
- net G0: now reaches J1.16 (Pin_16)
- net G0: now also A2.6 (D3)
- net B0: now reaches J1.2 (Pin_2)
- net B0: now also A2.7 (D4)
- net R1: now reaches J1.3 (Pin_3)
- net R1: now also A2.8 (D5)
- net B1: now reaches J1.4 (Pin_4)
- net B1: now also A2.10 (D7)
- net RowA: now reaches J1.5 (Pin_5)
- net RowA: now also A2.19 (A0)
- net RowC: now reaches J1.6 (Pin_6)
- net RowC: now also A2.21 (A2)
- net CLK: now reaches J1.7 (Pin_7)
- net CLK: now also A2.11 (D8)
- net OE: now reaches J1.8 (Pin_8)
- net OE: now also A2.12 (D9)
- net at A1.28 (~{RESET}): now also A1.3 (~{RESET}), R15.2, SW1.1
Other:
- title: (none) -> PONG RGB LED Matrix
- moved on the sheet: C1, C2, D1, J1, J2

Commit message: Tidy up and commenting
Parts:
- RV1: value R_Potentiometer -> P1_Dial
- RV2: value R_Potentiometer -> P2_Dial
- SW1: value SW_Push -> Reset_Switch
- U3, U4: footprint Display_7Segment:HDSP-A151 -> Display_7Segment:D1X8K
Connections:
- net +5V: now also A2.27 (+5V)
- net B0: now also J1.3; no longer J1.2 (Pin_2)
- net B1: now also J1.7 (Pin_4); no longer J1.4 (Pin_4)
- net CLK: now also J1.13 (Pin_7); no longer J1.7 (Pin_7)
- net G0: now also J1.2 (Pin_16); no longer J1.16 (Pin_16)
- net G1: now also J1.6 (Pin_14); no longer J1.14 (Pin_14)
- net GND: now also J1.12 (Pin_11), J1.16 (Pin_9), J1.4 (Pin_15), J1.8 (Pin_13), U3.3 (CA), U3.8 (CA), U4.3 (CA), U4.8 (CA); no longer J1.11 (Pin_11), J1.13 (Pin_13), J1.15 (Pin_15), J1.9 (Pin_9), U3.1 (CA), U3.6 (CA), U4.1 (CA), U4.6 (CA)
- net LAT: now also J1.14 (Pin_10); no longer J1.10 (Pin_10)
- net OE: now also J1.15 (Pin_8); no longer J1.8 (Pin_8)
- net R1: now also J1.5 (Pin_3); no longer J1.3 (Pin_3)
- net RowA: now also J1.9 (Pin_5); no longer J1.5 (Pin_5)
- net RowB: now also J1.10 (Pin_12); no longer J1.12 (Pin_12)
- net RowC: now also J1.11 (Pin_6); no longer J1.6 (Pin_6)
- net at R9.2: now also U4.6 (B); no longer U4.9 (B)
- net at A1.3 (~{RESET}), R15.2, SW1.1: no longer A1.28 (~{RESET})
- net at R7.2: now also U3.10 (G); no longer U3.3 (G)
- net at R8.2: now also U4.7 (A); no longer U4.10 (A)
- net at R13.2: now also U4.9 (F); no longer U4.2 (F)
- net at R14.2: now also U4.10 (G); no longer U4.3 (G)
- net at R12.2: now also U4.1 (E); no longer U4.4 (E)
- net at R11.2: now also U4.2 (D); no longer U4.5 (D)
- net at R10.2: now also U4.4 (C); no longer U4.8 (C)
- net at R1.2: now also U3.7 (A); no longer U3.10 (A)
- net at U3.2 (D): now also R4.2; no longer R6.2
- net at R5.2: now also U3.1 (E); no longer U3.4 (E)
- net at U3.5 (DP): no longer R4.2
- net at R3.2: now also U3.4 (C); no longer U3.8 (C)
- net at R2.2: now also U3.6 (B); no longer U3.9 (B)
- new net: R6.2, U3.9 (F)
